File: kicad/Stopwatch/Stopwatch.kicad_sch (KiCad schematic)
At the start: 15 parts, among them SW1 SW_Push, U1 74HC14, U2 BluePill, U3 SC56-11GWA, U4 SC56-11GWA, U5 SC56-11GWA, U6 SC56-11GWA

Commit message: fixed BluePill symbol pin numbers, added button and BluePill footprint
Parts:
- C1, C2: footprint (none) -> Capacitor_THT:C_Disc_D3.0mm_W2.0mm_P2.50mm
- R1, R2, R3, R4, R5, R6: footprint (none) -> Resistor_THT:R_Axial_DIN0207_L6.3mm_D2.5mm_P10.16mm_Horizontal
- SW1: footprint (none) -> Custom:5ETH935
- U1: footprint (none) -> Package_DIP:DIP-14_W7.62mm
- U1: value (none) -> 74HC14; footprint (none) -> Package_DIP:DIP-14_W7.62mm
- U2: value BluePill -> (none)
- U3, U4, U5, U6: footprint (none) -> Custom:SC56-11GWA
Changed lines of the file:
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@@
     (property "Reference" "U1" (id 0) (at 106.68 166.37 0))
     (property "Value" "74HC14" (id 1) (at 106.68 168.91 0))
-    (property "Footprint" "" (id 2) (at 106.68 175.26 0)
+    (property "Footprint" "Package_DIP:DIP-14_W7.62mm" (id 2) (at 106.68 175.26 0)
       (effects (font (size 1.27 1.27)) hide)
     )
@@
       (effects (font (size 1.27 1.27)) (justify left))
     )
-    (property "Footprint" "" (id 2) (at 168.6052 205.74 0)
+    (property "Footprint" "Capacitor_THT:C_Disc_D3.0mm_W2.0mm_P2.50mm" (id 2) (at 168.6052 205.74 0)
       (effects (font (size 1.27 1.27)) hide)
     )
@@
     (property "Reference" "U3" (id 0) (at 217.17 60.96 0))
     (property "Value" "SC56-11GWA" (id 1) (at 217.17 63.5 0))
-    (property "Footprint" "" (id 2) (at 217.17 78.74 0)
+    (property "Footprint" "Custom:SC56-11GWA" (id 2) (at 217.17 78.74 0)
       (effects (font (size 1.27 1.27)) hide)
     )
@@
       (effects (font (size 1.27 1.27)) (justify left))
     )
-    (property "Footprint" "" (id 2) (at 35.2552 196.85 0)
+    (property "Footprint" "Capacitor_THT:C_Disc_D3.0mm_W2.0mm_P2.50mm" (id 2) (at 35.2552 196.85 0)
       (effects (font (size 1.27 1.27)) hide)
     )
@@
     (property "Reference" "U4" (id 0) (at 266.7 60.96 0))
     (property "Value" "SC56-11GWA" (id 1) (at 266.7 63.5 0))
-    (property "Footprint" "" (id 2) (at 266.7 78.74 0)
+    (property "Footprint" "Custom:SC56-11GWA" (id 2) (at 266.7 78.74 0)
       (effects (font (size 1.27 1.27)) hide)
     )
@@
     (property "Reference" "U5" (id 0) (at 316.23 60.96 0))
     (property "Value" "SC56-11GWA" (id 1) (at 316.23 63.5 0))
-    (property "Footprint" "" (id 2) (at 316.23 78.74 0)
+    (property "Footprint" "Custom:SC56-11GWA" (id 2) (at 316.23 78.74 0)
       (effects (font (size 1.27 1.27)) hide)
     )
@@
     (property "Reference" "R5" (id 0) (at 316.23 101.6 90))
     (property "Value" "120" (id 1) (at 316.23 99.06 90))
-    (property "Footprint" "" (id 2) (at 316.23 93.472 90)
+    (property "Footprint" "Resistor_THT:R_Axial_DIN0207_L6.3mm_D2.5mm_P10.16mm_Horizontal" (id 2) (at 316.23 93.472 90)
       (effects (font (size 1.27 1.27)) hide)
     )
@@
     (property "Reference" "R4" (id 0) (at 266.7 101.6 90))
     (property "Value" "120" (id 1) (at 266.7 99.06 90))
-    (property "Footprint" "" (id 2) (at 266.7 93.472 90)
+    (property "Footprint" "Resistor_THT:R_Axial_DIN0207_L6.3mm_D2.5mm_P10.16mm_Horizontal" (id 2) (at 266.7 93.472 90)
       (effects (font (size 1.27 1.27)) hide)
     )
@@
     (property "Reference" "U6" (id 0) (at 365.76 60.96 0))
     (property "Value" "SC56-11GWA" (id 1) (at 365.76 63.5 0))
-    (property "Footprint" "" (id 2) (at 365.76 78.74 0)
+    (property "Footprint" "Custom:SC56-11GWA" (id 2) (at 365.76 78.74 0)
       (effects (font (size 1.27 1.27)) hide)
     )
@@
       (effects (font (size 1.27 1.27)) (justify right))
     )
-    (property "Footprint" "" (id 2) (at 135.89 201.93 0)
+    (property "Footprint" "Custom:5ETH935" (id 2) (at 135.89 201.93 0)
       (effects (font (size 1.27 1.27)) hide)
     )
@@
     (in_bom yes) (on_board yes) (fields_autoplaced)
     (property "Reference" "U1" (id 0) (at 80.01 195.58 0))
-    (property "Value" "" (id 1) (at 80.01 198.12 0))
-    (property "Footprint" "" (id 2) (at 80.01 204.47 0)
+    (property "Value" "74HC14" (id 1) (at 80.01 198.12 0))
+    (property "Footprint" "Package_DIP:DIP-14_W7.62mm" (id 2) (at 80.01 204.47 0)
       (effects (font (size 1.27 1.27)) hide)
     )
@@
       (effects (font (size 1.27 1.27)) (justify left))
     )
-    (property "Value" "BluePill" (id 1) (at 95.25 83.82 0)
+    (property "Value" "" (id 1) (at 95.25 83.82 0)
       (effects (font (size 1.27 1.27)) (justify left))
     )
@@
     (pin "3")
     (pin "30")
-    (pin "30")
     (pin "31")
     (pin "32")
@@
     (pin "34")
     (pin "35")
+    (pin "36")
     (pin "37")
     (pin "38")
@@
       (effects (font (size 1.27 1.27)) (justify left))
     )
-    (property "Footprint" "" (id 2) (at 139.192 180.34 90)
+    (property "Footprint" "Resistor_THT:R_Axial_DIN0207_L6.3mm_D2.5mm_P10.16mm_Horizontal" (id 2) (at 139.192 180.34 90)
       (effects (font (size 1.27 1.27)) hide)
     )
@@
     (property "Reference" "U1" (id 0) (at 106.68 180.34 0))
     (property "Value" "74HC14" (id 1) (at 106.68 182.88 0))
-    (property "Footprint" "" (id 2) (at 106.68 189.23 0)
+    (property "Footprint" "Package_DIP:DIP-14_W7.62mm" (id 2) (at 106.68 189.23 0)
       (effects (font (size 1.27 1.27)) hide)
     )
@@
     (in_bom yes) (on_board yes) (fields_autoplaced)
     (property "Reference" "U1" (id 0) (at 80.01 180.34 0))
-    (property "Value" "" (id 1) (at 80.01 182.88 0))
-    (property "Footprint" "" (id 2) (at 80.01 189.23 0)
+    (property "Value" "74HC14" (id 1) (at 80.01 182.88 0))
+    (property "Footprint" "Package_DIP:DIP-14_W7.62mm" (id 2) (at 80.01 189.23 0)
       (effects (font (size 1.27 1.27)) hide)
     )
@@
     (property "Reference" "R3" (id 0) (at 217.17 101.6 90))
     (property "Value" "120" (id 1) (at 217.17 99.06 90))
-    (property "Footprint" "" (id 2) (at 217.17 93.472 90)
+    (property "Footprint" "Resistor_THT:R_Axial_DIN0207_L6.3mm_D2.5mm_P10.16mm_Horizontal" (id 2) (at 217.17 93.472 90)
       (effects (font (size 1.27 1.27)) hide)
     )
@@
     (property "Reference" "U1" (id 0) (at 106.68 195.58 0))
     (property "Value" "74HC14" (id 1) (at 106.68 198.12 0))
-    (property "Footprint" "" (id 2) (at 106.68 204.47 0)
+    (property "Footprint" "Package_DIP:DIP-14_W7.62mm" (id 2) (at 106.68 204.47 0)
       (effects (font (size 1.27 1.27)) hide)
     )
@@
     (property "Reference" "R6" (id 0) (at 365.76 101.6 90))
     (property "Value" "120" (id 1) (at 365.76 99.06 90))
-    (property "Footprint" "" (id 2) (at 365.76 93.472 90)
+    (property "Footprint" "Resistor_THT:R_Axial_DIN0207_L6.3mm_D2.5mm_P10.16mm_Horizontal" (id 2) (at 365.76 93.472 90)
       (effects (font (size 1.27 1.27)) hide)
     )
@@
       (effects (font (size 1.27 1.27)) (justify left))
     )
-    (property "Footprint" "" (id 2) (at 49.53 193.04 0)
+    (property "Footprint" "Package_DIP:DIP-14_W7.62mm" (id 2) (at 49.53 193.04 0)
       (effects (font (size 1.27 1.27)) hide)
     )
@@
     (property "Reference" "U1" (id 0) (at 180.34 184.15 0))
     (property "Value" "74HC14" (id 1) (at 180.34 186.69 0))
-    (property "Footprint" "" (id 2) (at 180.34 193.04 0)
+    (property "Footprint" "Package_DIP:DIP-14_W7.62mm" (id 2) (at 180.34 193.04 0)
       (effects (font (size 1.27 1.27)) hide)
     )
@@
     (property "Reference" "R2" (id 0) (at 156.21 199.39 90))
     (property "Value" "220k" (id 1) (at 156.21 196.85 90))
-    (property "Footprint" "" (id 2) (at 156.21 191.262 90)
+    (property "Footprint" "Resistor_THT:R_Axial_DIN0207_L6.3mm_D2.5mm_P10.16mm_Horizontal" (id 2) (at 156.21 191.262 90)
       (effects (font (size 1.27 1.27)) hide)
     )
@@
     )
     (path "/70939d1a-eebc-4600-a824-1ffc5bb21a58"
-      (reference "SW1") (unit 1) (value "SW_Push") (footprint "")
+      (reference "SW1") (unit 1) (value "SW_Push") (footprint "Custom:5ETH935")
     )
     (path "/e80ec6d0-5363-4b2e-8f69-84d8ce4e7c48"
@@
     )
     (path "/8fbc5cbb-84f9-4256-b3ca-01d837c9a331"
-      (reference "U2") (unit 1) (value "BluePill") (footprint "")
+      (reference "U2") (unit 1) (value "BluePill") (footprint "Custom:BluePill")
     )
     (path "/114a7b61-9a55-4ae0-8273-52f581c0e08b"
